Commit message: chore: remove unused URDF frames

File: models/ur_description/urdf/ur3e_cylinders_collision.urdf (robot description, URDF)
Before this commit: robot ur3e, 10 links, 9 joints
Links:
- removed link ur_base
- removed link ur_tool0
Joints:
- removed joint ur_base_link-base_fixed_joint
- removed joint ur_wrist_3_link-tool0_fixed_joint
